File: hardware/motorController.kicad_pcb (KiCad board)
At the start: 2 copper layers, 48.8 x 38 mm, 31 parts, among them J1 CONN_14X1, M1 Mounting Hole, M2 Mounting Hole, M3 Mounting Hole, M4 Mounting Hole, P1 CONN_1, P2 CONN_1, P3 CONN_1, P4 CONN_1, Q1 MOSFET-N, U1 7408, U2 MC33926

Commit message: silk
Other:
- board text added: "EN"
- board text added: "FB"
- board text added: "FWD"
- board text added: "GND"
- board text added: "IN1"
- board text added: "IN2"
- board text added: "INV"
- board text added: "MDIR"
- board text added: "MPWM"
- board text added: "OUT1"
- board text added: "OUT2"
- board text added: "POWER"
- board text added: "REV"
- board text added: "SF"
- board text added: "SLEW"
- board text added: "VCC"
- board text added: "VIN"
- board text added: "~D1"
- board text added: "~D2"
